File: PCB/Aioli/Aioli.kicad_pcb (KiCad board)
At the start: 2 copper layers, 57.1 x 58.7 mm, 46 parts, among them J1 USB_C_Receptacle_USB2.0, SW1 Rotary_Encoder_Switch, SW10 SW_Push, SW2 Rotary_Encoder_Switch, SW3 Rotary_Encoder_Switch, SW4 Rotary_Encoder_Switch, SW5 Rotary_Encoder_Switch, SW6 Rotary_Encoder_Switch, SW7 Rotary_Encoder_Switch, SW8 Rotary_Encoder_Switch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

Commit message: Generated Gerbers, CAD files
Other:
- net class Default removed
